File: freqcount_v2.0/Teiler_1Hz.kicad_sch (KiCad schematic)
At the start: 6 parts, among them J1 Conn_01x03_Male, U1 74LS390, U2 74LS390, U3 74LS390, U4 74LS390

Commit message: update
Parts:
- added J5: Conn_Coaxial, Connector_Coaxial:SMA_Amphenol_901-144_Vertical, symbol Connector:Conn_Coaxial
Connections:
- net 10MHz_Referenz: now also J5.1 (In)
- net GND: now also J5.2 (Ext)
Changed lines of the file:
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@@
   (junction (at 44.45 39.37) (diameter 0) (color 0 0 0 0)
+  )
+  (junction (at 60.96 39.37) (diameter 0) (color 0 0 0 0)
   )
   (no_connect (at 69.85 138.43))
@@
     (stroke (width 0) (type default) (color 0 0 0 0))
   )
+  (wire (pts (xy 60.96 39.37) (xy 60.96 45.72))
+    (stroke (width 0) (type default) (color 0 0 0 0))
+  )
   (wire (pts (xy 44.45 31.75) (xy 44.45 36.83))
     (stroke (width 0) (type default) (color 0 0 0 0))
   )
+  (wire (pts (xy 60.96 39.37) (xy 67.31 39.37))
+    (stroke (width 0) (type default) (color 0 0 0 0))
+  )
   (wire (pts (xy 76.2 48.26) (xy 107.95 48.26))
     (stroke (width 0) (type default) (color 0 0 0 0))
@@
     (stroke (width 0) (type default) (color 0 0 0 0))
   )
-  (wire (pts (xy 44.45 39.37) (xy 67.31 39.37))
+  (wire (pts (xy 44.45 39.37) (xy 60.96 39.37))
     (stroke (width 0) (type default) (color 0 0 0 0))
   )
@@
     )
     (pin "1")
+  )
+  (symbol (lib_id "Connector:Conn_Coaxial") (at 66.04 45.72 0) (unit 1)
+    (in_bom yes) (on_board yes)
+    (property "Reference" "J5" (id 0) (at 68.58 44.7431 0)
+      (effects (font (size 1.27 1.27)) (justify left))
+    )
+    (property "Value" "Conn_Coaxial" (id 1) (at 68.58 46.355 0)
+      (effects (font (size 1.27 1.27)) (justify left))
+    )
+    (property "Footprint" "Connector_Coaxial:SMA_Amphenol_901-144_Vertical" (id 2) (at 66.04 45.72 0)
+      (effects (font (size 1.27 1.27)) hide)
+    )
+    (property "Datasheet" " ~" (id 3) (at 66.04 45.72 0)
+      (effects (font (size 1.27 1.27)) hide)
+    )
+    (pin "1")
+    (pin "2")
   )
   (symbol (lib_id "power:GND") (at 44.45 93.98 0) (unit 1)
@@
     (pin "8")
   )
+  (symbol (lib_id "power:GND") (at 66.04 50.8 0) (unit 1)
+    (in_bom yes) (on_board yes)
+    (property "Reference" "#PWR028" (id 0) (at 66.04 57.15 0)
+      (effects (font (size 1.27 1.27)) hide)
+    )
+    (property "Value" "GND" (id 1) (at 69.215 52.705 0))
+    (property "Footprint" "" (id 2) (at 66.04 50.8 0)
+      (effects (font (size 1.27 1.27)) hide)
+    )
+    (property "Datasheet" "" (id 3) (at 66.04 50.8 0)
+      (effects (font (size 1.27 1.27)) hide)
+    )
+    (pin "1")
+  )
   (symbol (lib_id "power:GND") (at 175.26 63.5 0) (unit 1)
