File: freqcount_v2.0/freqcount1.1.kicad_sch (KiCad schematic)
At the start: 0 parts

Commit message: update
Other:
- added sheet hf_eingang (hf_eingang.kicad_sch)
- sheet Zaehler_Messsignal ports: added Messsignal; removed none
